File: PCB/ItsyBitsy breadboard.kicad_pcb (KiCad board)
At the start: 2 copper layers, 61 x 22.9 mm, 12 parts, among them J1 EDGE PINS, J2 EDGE PINS, J3 STEMMA_VOLTS, J4 STEMMA, J5 BATTERY, J6 XTRA, J7 BODGE PINS, J8 EDGE PINS

Commit message: update with new design and photos
Parts:
- removed J3: STEMMA_VOLTS, Adafruit:Pin_Header_Straight_1x03_Pitch2.54mm_no_silk
- removed the REF** at (163.1, 116.5)
- removed the REF** at (163.1, 99.4)
- added C1: 10uF, Capacitors_SMD:C_0805, F.Cu at (107.6, 102.9)
- added D1: CHARGE, LEDs:LED_0805, F.Cu at (104.3, 104.0)
- added D2: PWR, LEDs:LED_0805, F.Cu at (104.3, 116.5)
- added JMP1: SCL_RX, Connectors:GS3, B.Cu at (133.7, 104.9)
- added JMP2: SDA_TX, Connectors:GS3, B.Cu at (139.7, 104.9)
- added JMP3: Vbat -> A6, Connectors:GS2, B.Cu at (128.4, 111.8)
- added JMP4: STEMMA_VOLTS, Connectors:GS3, B.Cu at (149.0, 107.1)
- added Q1: BSS138DW-7-F, digikey-footprints:SOT-363, F.Cu at (135.7, 109.8)
- added R1: 1K, Resistors_SMD:R_0805, F.Cu at (110.7, 108.6)
- added R2: 1.5K, Resistors_SMD:R_0805, F.Cu at (106.6, 116.1)
- added R3: 100K, Resistors_SMD:R_0805, F.Cu at (113.7, 106.9)
- added R4: 10K, Resistors_SMD:R_0805, F.Cu at (107.7, 109.2)
- added R5: 100K, Resistors_SMD:R_0805, F.Cu at (113.7, 109.2)
- added REF**: MountingHole_2.7mm_M2.5, Mounting_Holes:MountingHole_2.7mm_M2.5, F.Cu at (157.5, 116.5)
- added REF**: MountingHole_2.7mm_M2.5, Mounting_Holes:MountingHole_2.7mm_M2.5, F.Cu at (157.5, 99.4)
- added RN1: 4x10K, Resistors_SMD:R_Array_Convex_4x0603, F.Cu at (139.0, 109.9)
- added U1: MCP73831-2-OT, TO_SOT_Packages_SMD:SOT-23-5, F.Cu at (107.4, 106.0)
- moved J5 50.8 mm to (106.8, 99.3), turned to 180 degrees
- moved REF** 8.13 mm to (99.3, 99.4)
- moved REF** 8.13 mm to (99.3, 116.5)
- moved J4 6.43 mm to (152.4, 111.0)
Connections:
- net /RST renamed /~RST
- J4 pad 1: /SCL -> /STEMMA_SCL
- J4 pad 2: /SDA -> /STEMMA_SDA
Routing:
- net /Vhi: track 2.54 -> 71.3 mm, vias 0 -> 3
- net +5V: track 42.1 -> 2.54 mm
- net /BAT: track 51.0 -> 20.4 mm, vias 1 -> 0
- net /STEMMA_SCL: track 0.00 -> 23.8 mm
- net /STEMMA_SDA: track 0.00 -> 23.2 mm
- net /SCL: track 34.1 -> 11.1 mm, vias 2 -> 1
- net /SDA: track 29.3 -> 7.64 mm, vias 0 -> 1
- net /SCL_RX: track 0.00 -> 20.6 mm, vias 0 -> 2
- net /D2-A6: track 2.54 -> 21.8 mm, vias 0 -> 1
- net Net-(JMP3-Pad2): track 0.00 -> 18.1 mm, vias 0 -> 1
- net Net-(J4-Pad3): track 7.43 -> 24.5 mm, vias 0 -> 1
- net /SDA_TX: track 0.00 -> 14.8 mm, vias 0 -> 2
- net +3V3: track 47.1 -> 61.7 mm, vias 0 -> 1
- net /D0-RX: track 2.54 -> 16.3 mm, vias 0 -> 1
- net Net-(D1-Pad1): track 0.00 -> 13.5 mm
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Other:
- board size 61 x 22.9 mm -> 63.5 x 22.9 mm
- board text added: "+"
- board text added: "2.5 in x 0.9 in M2.5 mounting holes"
- board text added: "2019-11-24 v02"
- board text added: "3.3v"
- board text added: "5v"
- board text added: "LiPo charge rate = 100mA"
- board text added: "RX SCL"
- board text added: "STEMMA CONNECTOR"
- board text added: "STEMMA DATA SOURCE"
- board text added: "TX SDA"
- board text removed: "+3.3v"
- board text removed: "+5v"
- board text removed: "2.4 in x 0.75 in; M2.5 mounting holes"
- board text removed: "2019-04-27 v01"
- board text removed: "A stacking breakout board to adapt the ItsyBitsy M4 Express for use with a standard breadboard or protoboard."
