File: PCB/ItsyBitsy breadboard.sch (KiCad schematic (older format))
At the start: 9 parts, among them J1 EDGE PINS, J2 EDGE PINS, J3 STEMMA_VOLTS, J4 STEMMA, J5 BATTERY, J6 XTRA, J7 BODGE PINS, J8 EDGE PINS, M1 ItsyBitsy_M4_Express

Commit message: update with new design and photos
Parts:
- removed J3: STEMMA_VOLTS, Adafruit:Pin_Header_Straight_1x03_Pitch2.54mm_no_silk, symbol conn:CONN_01X03
- added C1: 10uF, Capacitors_SMD:C_0805, symbol device:CP1_Small
- added D1: ORG, LEDs:LED_0805, symbol device:LED_Small
- added D2: GRN, LEDs:LED_0805, symbol device:LED_Small
- added JMP1: SCL_RX, Connectors:GS3, symbol conn:GS3
- added JMP2: SDA_TX, Connectors:GS3, symbol conn:GS3
- added JMP3: Vbat, Connectors:GS2, symbol conn:GS2
- added JMP4: STEMMA_VOLTS, Connectors:GS3, symbol conn:GS3
- added Q1: BSS138DW-7-F, digikey-footprints:SOT-363, symbol dk_Transistors-FETs-MOSFETs-Arrays:BSS138DW-7-F
- added R1: 1K, Resistors_SMD:R_0805, symbol device:R_Small
- added R2: 1.5K, Resistors_SMD:R_0805, symbol device:R_Small
- added R3, R5: 100K, Resistors_SMD:R_0805, symbol device:R_Small
- added R4: 10K, Resistors_SMD:R_0805, symbol device:R_Small
- added RN1: 4x10K, Resistors_SMD:R_Array_Convex_4x0603, symbol device:R_Pack04
- added U1: MCP73831-2-OT, TO_SOT_Packages_SMD:SOT-23-5, symbol battery_management:MCP73831-2-OT
Connections:
- net labels added: SCL_RX, SDA_TX, STEMMA_SCL, STEMMA_SDA, ~RST
- net labels removed: RST
- wire segments 139 -> 214
Other:
- note added: "100mA\nCHARGE\nRATE"
- note added: "BATTERY MANAGEMENT"
- note added: "POWER"
- note removed: "STEMMA Voltage\nSelect Jumper"

Commit message: Update STEMMA type default
Connections:
- net labels added: +V
- wire segments 214 -> 220
Other:
- note added: "Defaults to +3.3V"
Changed lines of the file:
@@
 Wire Wire Line
 	8275 5325 8400 5325
-Wire Wire Line
-	8275 5225 8400 5225
 $Comp
 L conn:CONN_01X16 J2
@@
 Wire Wire Line
 	7225 5625 7350 5625
-Text Label 7750 5025 0    50   ~ 0
+Text Label 7950 5025 0    50   ~ 0
 STEMMA_SCL
-Text Label 7750 5125 0    50   ~ 0
+Text Label 7950 5125 0    50   ~ 0
 STEMMA_SDA
 Text Label 5575 5025 0    50   ~ 0
@@
 Wire Wire Line
 	6100 5325 6100 4650
-Wire Wire Line
-	7550 5125 8400 5125
 Wire Wire Line
 	6100 5950 7550 5950
@@
 $EndComp
 Wire Wire Line
-	7650 5025 8400 5025
-Wire Wire Line
 	8375 3925 8375 3750
-Wire Wire Line
-	8275 4350 8275 5225
 Wire Wire Line
 	8175 3825 8175 3850
@@
 Wire Wire Line
 	8275 4225 8275 4350
-Connection ~ 8275 4350
-Wire Wire Line
-	6725 3850 8175 3850
-Wire Wire Line
-	7250 4350 8275 4350
+Wire Wire Line
+	6725 3850 8050 3850
 Wire Wire Line
 	6825 3925 7250 3925
@@
 Connection ~ 6100 4650
 Connection ~ 6625 3850
+Wire Wire Line
+	7750 5225 8400 5225
+Wire Wire Line
+	7250 4350 7750 4350
+Wire Wire Line
+	7750 5225 7750 5125
+Connection ~ 7750 4350
+Wire Wire Line
+	7750 4350 8050 4350
+Wire Wire Line
+	7750 5025 7750 4350
+Wire Wire Line
+	7750 5125 7750 5025
+Wire Wire Line
+	7650 5025 8400 5025
+Wire Wire Line
+	7550 5125 8400 5125
+Text Label 8125 4350 0    50   ~ 0
++V
+Wire Wire Line
+	8050 4350 8050 3850
+Connection ~ 8050 4350
+Wire Wire Line
+	8050 4350 8275 4350
+Connection ~ 8050 3850
+Wire Wire Line
+	8050 3850 8175 3850
+Text Notes 8425 4325 0    50   ~ 0
+Defaults to +3.3V
 $EndSCHEMATC

Commit message: update charging design
Connections:
- net labels removed: +5V
- wire segments 220 -> 219
Changed lines of the file:
@@
 	5200 1250 5750 1250
-Wire Wire Line
-	5875 1450 5875 925
-Wire Wire Line
-	5200 1450 5875 1450
 Wire Wire Line
 	4500 3000 4500 3300
@@
 Text Notes 4550 6750 0    50   ~ 0
 Battery
-$Comp
-L power:+5V #PWR0101
-U 1 1 5CDD68C7
-P 5875 925
-F 0 "#PWR0101" H 5875 775 50  0001 C CNN
-F 1 "+5V" H 5890 1098 50  0000 C CNN
-F 2 "" H 5875 925 50  0001 C CNN
-F 3 "" H 5875 925 50  0001 C CNN
-	1    5875 925
-	1    0    0    -1
-$EndComp
 $Comp
 L conn:CONN_01X05 J6
@@
 Wire Wire Line
 	2850 6175 2500 6175
-Text Label 2500 6175 0    50   ~ 0
-Vhi
 $Comp
 L device:R_Small R4
@@
 Text Notes 8425 4325 0    50   ~ 0
 Defaults to +3.3V
+Wire Wire Line
+	5200 1450 5750 1450
+Text Label 2500 6175 2    50   ~ 0
+USB
 $EndSCHEMATC

Commit message: update charging LED resistor
Parts:
- R1: value 1K -> 1.5K
Changed lines of the file:
@@
 P 3350 6375
 F 0 "R1" H 3409 6421 50  0000 L CNN
-F 1 "1K" H 3409 6330 50  0000 L CNN
+F 1 "1.5K" H 3409 6330 50  0000 L CNN
 F 2 "Resistors_SMD:R_0805" H 3350 6375 50  0001 C CNN
 F 3 "" H 3350 6375 50  0001 C CNN

Commit message: add default Stemma jumpers
Connections:
- wire segments 219 -> 229
Changed lines of the file:
@@
 $EndComp
 Wire Wire Line
-	5150 4925 4750 4925
+	5150 4925 4950 4925
 Text Label 4750 4925 0    50   ~ 0
 SCL
@@
 	5150 5125 4750 5125
 Wire Wire Line
-	5150 5450 4750 5450
+	5150 5450 4950 5450
 Text Label 4750 5450 0    50   ~ 0
 SDA
@@
 D0-RX
 Wire Wire Line
-	5450 5550 5900 5550
-Wire Wire Line
 	5900 5550 5900 6025
 Wire Wire Line
 	7225 5025 7650 5025
 Wire Wire Line
-	5450 5025 6000 5025
+	5450 5025 5550 5025
 Wire Wire Line
 	6525 3925 6525 3975
@@
 Text Label 2500 6175 2    50   ~ 0
 USB
+Wire Wire Line
+	4950 4925 4950 4625
+Wire Wire Line
+	4950 4625 5550 4625
+Wire Wire Line
+	5550 4625 5550 5025
+Connection ~ 4950 4925
+Wire Wire Line
+	4950 4925 4750 4925
+Connection ~ 5550 5025
+Wire Wire Line
+	5550 5025 6000 5025
+Wire Wire Line
+	4950 5450 4950 5300
+Wire Wire Line
+	4950 5300 5550 5300
+Wire Wire Line
+	5550 5300 5550 5550
+Wire Wire Line
+	5450 5550 5550 5550
+Connection ~ 4950 5450
+Wire Wire Line
+	4950 5450 4750 5450
+Connection ~ 5550 5550
+Wire Wire Line
+	5550 5550 5900 5550
 $EndSCHEMATC
